File: Dashboard-module/Hardware/PCB/Dashboard.kicad_sch (KiCad schematic)
At the start: 84 parts, among them IC1 ATA6563-GAQW1, IC2 MCP16361T-E_NMX, J1 F31L-1A7H1-11030, J2 DM3CS-SF, J3 DT15-12PA, Q1 BC850, Q2 BC850, U1 SN65HVD230, U5 MIC29301

Commit message: feature: Add latest docs
Connections:
- net 3V3: now also R1.1, R15.1
- net 5V: now also LED1.1 (A_1), LED1.A1 (A_2), LED2.1 (A_1), LED2.A1 (A_2); no longer LED1.2 (K_1), LED1.A2 (K_2), LED2.2 (K_1), LED2.A2 (K_2), R1.1, R15.1
- new net: LED2.2 (K_1), LED2.A2 (K_2), R32.1
- new net: LED1.2 (K_1), LED1.A2 (K_2), R21.1
Other:
- moved on the sheet: LED1
