File: Dashboard-module/Hardware/PCB/esp32-integration.kicad_sch (KiCad schematic)
At the start: 37 parts, among them J6 USB4800-03-A, Q3 BC850, Q4 BC850, SW5 boot_button, SW6 boot_button, U2 ESP32-WROOM-32, U3 CP2102-GMR, U4 MPU-6050

Commit message: feature: Add latest docs
Parts:
- removed C10: 0.1uF, Capacitor_SMD:C_1210_3225Metric_Pad1.33x2.70mm_HandSolder, symbol Device:C
- removed C13: 0.1uF, Capacitor_SMD:C_1210_3225Metric_Pad1.33x2.70mm_HandSolder, symbol Device:C_Small
Other:
- note removed: "C10 as debounce"
